Commit message: 带臂&比赛地形

File: resources/robots/SF_TRON1A/urdf/robo.urdf (robot description, URDF)
Before this commit: robot SF_TRON1, 10 links, 9 joints
Links:
- added link airbot_arm, mass 0.77705; visual mesh filename=/home/qi/limx_rl/pointfoot-legged-gym/resources/robots/SF_T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
- added link airbot_arm_base, mass 0.17; visual box size=0.15 0.15 0.006
- added link link1, mass 0.5571; visual mesh filename=/home/qi/limx_rl/pointfoot-legged-gym/resources/robots/SF_T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
- added link link2, mass 0.64621; collision box size=0.2 0.04 0.04; visual mesh filename=/home/qi/limx_rl/pointfoot-legged-gym/resources/robots/SF_T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
- added link link3, mass 0.28804; collision box size=0.04 0.35 0.04; visual mesh filename=/home/qi/limx_rl/pointfoot-legged-gym/resources/robots/SF_T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
- added link link4, mass 0.34876; visual mesh filename=/home/qi/limx_rl/pointfoot-legged-gym/resources/robots/SF_T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
- added link link5, mass 0.36132; visual mesh filename=/home/qi/limx_rl/pointfoot-legged-gym/resources/robots/SF_T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
- added link link6, mass 0.65361; collision box size=0.08 0.04 0.1; visual mesh filename=/home/qi/limx_rl/pointfoot-legged-gym/resources/robots/SF_T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
- link abad_L_Link: geometry collision cylinder length=0.05 radius=0.05; visual mesh filename=/home/qi/limx_rl/pointfoot-legged-gym/resources/robots/SF_T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
- link abad_R_Link: geometry collision cylinder length=0.05 radius=0.05; visual mesh filename=/home/qi/limx_rl/pointfoot-legged-gym/resources/robots/SF_T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
- link ankle_L_Link: geometry collision mesh filename=/home/qi/limx_rl/pointfoot-legged-gym/resources/robots/SF_T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; visual mesh filename=/home/qi/limx_rl/pointfoot-legged-gym/resources/robots/SF_T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
- link ankle_R_Link: geometry collision mesh filename=/home/qi/limx_rl/pointfoot-legged-gym/resources/robots/SF_T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; visual mesh filename=/home/qi/limx_rl/pointfoot-legged-gym/resources/robots/SF_T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
- link base_Link: geometry collision box size=0.27 0.26 0.19; visual mesh filename=/home/qi/limx_rl/pointfoot-legged-gym/resources/robots/SF_T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
- link hip_L_Link: geometry collision cylinder length=0.15 radius=0.035; visual mesh filename=/home/qi/limx_rl/pointfoot-legged-gym/resources/robots/SF_T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
- link hip_R_Link: geometry collision cylinder length=0.15 radius=0.035; visual mesh filename=/home/qi/limx_rl/pointfoot-legged-gym/resources/robots/SF_T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
- link knee_L_Link: geometry collision cylinder length=0.26 radius=0.02; visual mesh filename=/home/qi/limx_rl/pointfoot-legged-gym/resources/robots/SF_T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
- link knee_R_Link: geometry collision cylinder length=0.26 radius=0.02; visual mesh filename=/home/qi/limx_rl/pointfoot-legged-gym/resources/robots/SF_T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
Joints:
- added joint J1: type fixed, parent airbot_arm, child link1, origin xyz=0 0 0.1172 rpy=0 0 0
- added joint J2: type fixed, parent link1, child link2, origin xyz=0 0 0 rpy=1.5708 -2.7549 0
- added joint J3: type fixed, parent link2, child link3, origin xyz=0.27009 0 0 rpy=0 0 1.9575
- added joint J4: type fixed, parent link3, child link4, origin xyz=0 0.30854 0 rpy=-1.5708 -1.5708 0
- added joint J5: type fixed, parent link4, child link5, origin xyz=0 0 0 rpy=1.5708 0 0
- added joint J6: type fixed, parent link5, child link6, origin xyz=0 0.26145 0 rpy=-1.5708 0 0
- added joint airbot_arm_base_joint: type fixed, parent base_Link, child airbot_arm_base, origin xyz=0.00166 0 0.0195 rpy=0. 0. 0.
- added joint airbot_arm_joint: type fixed, parent airbot_arm_base, child airbot_arm, origin xyz=0.0245 0. 0.003 rpy=0. 0. 0.
